Commit message: joint_idx for go finished

File: resources/robots/a1/urdf/a1.urdf (robot description, URDF)
Before this commit: robot a1_description, 23 links, 22 joints
Links:
- removed link FL_calf
- removed link FL_foot
- removed link FL_thigh
- removed link FL_thigh_shoulder
- removed link FR_calf
- removed link FR_foot
- removed link FR_thigh
- removed link FR_thigh_shoulder
- removed link RL_calf
- removed link RL_foot
- removed link RL_thigh
- removed link RL_thigh_shoulder
- removed link RR_calf
- removed link RR_foot
- removed link RR_thigh
- removed link RR_thigh_shoulder
- removed link base
- added link FL_lower, mass 0.166; collision box size=0.2 0.016 0.016; visual mesh filename=meshes/calf.obj scale=1 1 1
- added link FL_toe, mass 0.06; collision sphere radius=0.02; visual sphere radius=0.01
- added link FL_upper, mass 1.013; collision box size=0.2 0.0245 0.034; visual mesh filename=meshes/thigh.obj scale=1 1 1
- added link FR_lower, mass 0.166; collision box size=0.2 0.016 0.016; visual mesh filename=meshes/calf.obj scale=1 1 1
- added link FR_toe, mass 0.06; collision sphere radius=0.02; visual sphere radius=0.01
- added link FR_upper, mass 1.013; collision box size=0.2 0.0245 0.034; visual mesh filename=meshes/thigh_mirror.obj scale=1 1 1
- added link RL_lower, mass 0.166; collision box size=0.2 0.016 0.016; visual mesh filename=meshes/calf.obj scale=1 1 1
- added link RL_toe, mass 0.06; collision sphere radius=0.02; visual sphere radius=0.01
- added link RL_upper, mass 1.013; collision box size=0.2 0.0245 0.034; visual mesh filename=meshes/thigh.obj scale=1 1 1
- added link RR_lower, mass 0.166; collision box size=0.2 0.016 0.016; visual mesh filename=meshes/calf.obj scale=1 1 1
- added link RR_toe, mass 0.06; collision sphere radius=0.02; visual sphere radius=0.01
- added link RR_upper, mass 1.013; collision box size=0.2 0.0245 0.034; visual mesh filename=meshes/thigh_mirror.obj scale=1 1 1
- link FL_hip: geometry collision cylinder length=0.04 radius=0.046; visual mesh filename=meshes/hip.obj scale=1 1 1
- link FR_hip: geometry collision cylinder length=0.04 radius=0.046; visual mesh filename=meshes/hip.obj scale=1 1 1
- link RL_hip: geometry collision cylinder length=0.04 radius=0.046; visual mesh filename=meshes/hip.obj scale=1 1 1
- link RR_hip: geometry collision cylinder length=0.04 radius=0.046; visual mesh filename=meshes/hip.obj scale=1 1 1
- link imu_link: geometry collision box size=.001 .001 .001; visual box size=0.001 0.001 0.001
- link trunk: geometry collision box size=0.05 0.125 0.06; collision box size=0.267 0.194 0.114
Joints:
- removed joint floating_base
- removed joint leg0_FL_a_hip_joint
- removed joint leg0_FL_b_hip_fixed
- removed joint leg0_FL_c_thigh_joint
- removed joint leg0_FL_d_calf_joint
- removed joint leg0_FL_e_foot_fixed
- removed joint leg1_FR_a_hip_joint
- removed joint leg1_FR_b_hip_fixed
- removed joint leg1_FR_c_thigh_joint
- removed joint leg1_FR_d_calf_joint
- removed joint leg1_FR_e_foot_fixed
- removed joint leg2_RL_a_hip_joint
- removed joint leg2_RL_b_hip_fixed
- removed joint leg2_RL_c_thigh_joint
- removed joint leg2_RL_d_calf_joint
- removed joint leg2_RL_e_foot_fixed
- removed joint leg3_RR_a_hip_joint
- removed joint leg3_RR_b_hip_fixed
- removed joint leg3_RR_c_thigh_joint
- removed joint leg3_RR_d_calf_joint
- removed joint leg3_RR_e_foot_fixed
- added joint FL_hip_joint: type revolute, parent trunk, child FL_hip, origin xyz=0.183 0.047 0 rpy=0 0 0, axis 1 0 0, limit lower=-0.802851455917 upper=0.802851455917 effort=33.5 velocity=16
- added joint FL_lower_joint: type revolute, parent FL_upper, child FL_lower, origin xyz=0 0 -0.2 rpy=0 0 0, axis 0 1 0, limit lower=-2.69653369433 upper=-0.916297857297 effort=33.5 velocity=16
- added joint FL_toe_fixed: type fixed, parent FL_lower, child FL_toe, origin xyz=0 0 -0.2 rpy=0 0 0
- added joint FL_upper_joint: type revolute, parent FL_hip, child FL_upper, origin xyz=0 0.08505 0 rpy=0 0 0, axis 0 1 0, limit lower=-1.0471975512 upper=4.18879020479 effort=33.5 velocity=16
- added joint FR_hip_joint: type revolute, parent trunk, child FR_hip, origin xyz=0.183 -0.047 0 rpy=0 0 0, axis 1 0 0, limit lower=-0.802851455917 upper=0.802851455917 effort=33.5 velocity=16
- added joint FR_lower_joint: type revolute, parent FR_upper, child FR_lower, origin xyz=0 0 -0.2 rpy=0 0 0, axis 0 1 0, limit lower=-2.69653369433 upper=-0.916297857297 effort=33.5 velocity=16
- added joint FR_toe_fixed: type fixed, parent FR_lower, child FR_toe, origin xyz=0 0 -0.2 rpy=0 0 0
- added joint FR_upper_joint: type revolute, parent FR_hip, child FR_upper, origin xyz=0 -0.08505 0 rpy=0 0 0, axis 0 1 0, limit lower=-1.0471975512 upper=4.18879020479 effort=33.5 velocity=16
- added joint RL_hip_joint: type revolute, parent trunk, child RL_hip, origin xyz=-0.183 0.047 0 rpy=0 0 0, axis 1 0 0, limit lower=-0.802851455917 upper=0.802851455917 effort=33.5 velocity=16
- added joint RL_lower_joint: type revolute, parent RL_upper, child RL_lower, origin xyz=0 0 -0.2 rpy=0 0 0, axis 0 1 0, limit lower=-2.69653369433 upper=-0.916297857297 effort=33.5 velocity=16
- added joint RL_toe_fixed: type fixed, parent RL_lower, child RL_toe, origin xyz=0 0 -0.2 rpy=0 0 0
- added joint RL_upper_joint: type revolute, parent RL_hip, child RL_upper, origin xyz=0 0.08505 0 rpy=0 0 0, axis 0 1 0, limit lower=-1.0471975512 upper=4.18879020479 effort=33.5 velocity=16
- added joint RR_hip_joint: type revolute, parent trunk, child RR_hip, origin xyz=-0.183 -0.047 0 rpy=0 0 0, axis 1 0 0, limit lower=-0.802851455917 upper=0.802851455917 effort=33.5 velocity=16
- added joint RR_lower_joint: type revolute, parent RR_upper, child RR_lower, origin xyz=0 0 -0.2 rpy=0 0 0, axis 0 1 0, limit lower=-2.69653369433 upper=-0.916297857297 effort=33.5 velocity=16
- added joint RR_toe_fixed: type fixed, parent RR_lower, child RR_toe, origin xyz=0 0 -0.2 rpy=0 0 0
- added joint RR_upper_joint: type revolute, parent RR_hip, child RR_upper, origin xyz=0 -0.08505 0 rpy=0 0 0, axis 0 1 0, limit lower=-1.0471975512 upper=4.18879020479 effort=33.5 velocity=16

Commit message: a1 fixed

File: resources/robots/a1/urdf/a1.urdf (robot description, URDF)
Before this commit: robot a1_description, 19 links, 18 joints
Links:
- removed link FL_lower
- removed link FL_toe
- removed link FL_upper
- removed link FR_lower
- removed link FR_toe
- removed link FR_upper
- removed link RL_lower
- removed link RL_toe
- removed link RL_upper
- removed link RR_lower
- removed link RR_toe
- removed link RR_upper
- added link FL_calf, mass 0.166; collision box size=0.2 0.016 0.016; visual mesh filename=../meshes/calf.dae scale=1 1 1
- added link FL_foot, mass 0.06; collision sphere radius=0.02; visual sphere radius=0.01
- added link FL_thigh, mass 1.013; collision box size=0.2 0.0245 0.034; visual mesh filename=../meshes/thigh.dae scale=1 1 1
- added link FL_thigh_shoulder
- added link FR_calf, mass 0.166; collision box size=0.2 0.016 0.016; visual mesh filename=../meshes/calf.dae scale=1 1 1
- added link FR_foot, mass 0.06; collision sphere radius=0.02; visual sphere radius=0.01
- added link FR_thigh, mass 1.013; collision box size=0.2 0.0245 0.034; visual mesh filename=../meshes/thigh_mirror.dae scale=1 1 1
- added link FR_thigh_shoulder
- added link RL_calf, mass 0.166; collision box size=0.2 0.016 0.016; visual mesh filename=../meshes/calf.dae scale=1 1 1
- added link RL_foot, mass 0.06; collision sphere radius=0.02; visual sphere radius=0.01
- added link RL_thigh, mass 1.013; collision box size=0.2 0.0245 0.034; visual mesh filename=../meshes/thigh.dae scale=1 1 1
- added link RL_thigh_shoulder
- added link RR_calf, mass 0.166; collision box size=0.2 0.016 0.016; visual mesh filename=../meshes/calf.dae scale=1 1 1
- added link RR_foot, mass 0.06; collision sphere radius=0.02; visual sphere radius=0.01
- added link RR_thigh, mass 1.013; collision box size=0.2 0.0245 0.034; visual mesh filename=../meshes/thigh_mirror.dae scale=1 1 1
- added link RR_thigh_shoulder
- link FL_hip: geometry visual mesh filename=../meshes/hip.dae scale=1 1 1
- link FR_hip: geometry visual mesh filename=../meshes/hip.dae scale=1 1 1
- link RL_hip: geometry visual mesh filename=../meshes/hip.dae scale=1 1 1
- link RR_hip: geometry visual mesh filename=../meshes/hip.dae scale=1 1 1
- link imu_link: geometry visual box size=0.001 0.001 0.001
- link trunk: geometry collision box size=0.267 0.194 0.114; visual mesh filename=../meshes/trunk.dae scale=1 1 1
Joints:
- removed joint FL_lower_joint
- removed joint FL_toe_fixed
- removed joint FL_upper_joint
- removed joint FR_lower_joint
- removed joint FR_toe_fixed
- removed joint FR_upper_joint
- removed joint RL_lower_joint
- removed joint RL_toe_fixed
- removed joint RL_upper_joint
- removed joint RR_lower_joint
- removed joint RR_toe_fixed
- removed joint RR_upper_joint
- added joint FL_calf_joint: type revolute, parent FL_thigh, child FL_calf, origin xyz=0 0 -0.2 rpy=0 0 0, axis 0 1 0, limit lower=-2.69653369433 upper=-0.916297857297 effort=55 velocity=28.6
- added joint FL_foot_fixed: type fixed, parent FL_calf, child FL_foot, origin xyz=0 0 -0.2 rpy=0 0 0
- added joint FL_hip_fixed: type fixed, parent FL_hip, child FL_thigh_shoulder, origin xyz=0 0.081 0 rpy=0 0 0
- added joint FL_thigh_joint: type revolute, parent FL_hip, child FL_thigh, origin xyz=0 0.08505 0 rpy=0 0 0, axis 0 1 0, limit lower=-1.0471975512 upper=4.18879020479 effort=55 velocity=28.6
- added joint FR_calf_joint: type revolute, parent FR_thigh, child FR_calf, origin xyz=0 0 -0.2 rpy=0 0 0, axis 0 1 0, limit lower=-2.69653369433 upper=-0.916297857297 effort=55 velocity=28.6
- added joint FR_foot_fixed: type fixed, parent FR_calf, child FR_foot, origin xyz=0 0 -0.2 rpy=0 0 0
- added joint FR_hip_fixed: type fixed, parent FR_hip, child FR_thigh_shoulder, origin xyz=0 -0.081 0 rpy=0 0 0
- added joint FR_thigh_joint: type revolute, parent FR_hip, child FR_thigh, origin xyz=0 -0.08505 0 rpy=0 0 0, axis 0 1 0, limit lower=-1.0471975512 upper=4.18879020479 effort=55 velocity=28.6
- added joint RL_calf_joint: type revolute, parent RL_thigh, child RL_calf, origin xyz=0 0 -0.2 rpy=0 0 0, axis 0 1 0, limit lower=-2.69653369433 upper=-0.916297857297 effort=55 velocity=28.6
- added joint RL_foot_fixed: type fixed, parent RL_calf, child RL_foot, origin xyz=0 0 -0.2 rpy=0 0 0
- added joint RL_hip_fixed: type fixed, parent RL_hip, child RL_thigh_shoulder, origin xyz=0 0.081 0 rpy=0 0 0
- added joint RL_thigh_joint: type revolute, parent RL_hip, child RL_thigh, origin xyz=0 0.08505 0 rpy=0 0 0, axis 0 1 0, limit lower=-1.0471975512 upper=4.18879020479 effort=55 velocity=28.6
- added joint RR_calf_joint: type revolute, parent RR_thigh, child RR_calf, origin xyz=0 0 -0.2 rpy=0 0 0, axis 0 1 0, limit lower=-2.69653369433 upper=-0.916297857297 effort=55 velocity=28.6
- added joint RR_foot_fixed: type fixed, parent RR_calf, child RR_foot, origin xyz=0 0 -0.2 rpy=0 0 0
- added joint RR_hip_fixed: type fixed, parent RR_hip, child RR_thigh_shoulder, origin xyz=0 -0.081 0 rpy=0 0 0
- added joint RR_thigh_joint: type revolute, parent RR_hip, child RR_thigh, origin xyz=0 -0.08505 0 rpy=0 0 0, axis 0 1 0, limit lower=-1.0471975512 upper=4.18879020479 effort=55 velocity=28.6
- joint FL_hip_joint: limit lower=-0.802851455917 upper=0.802851455917 effort=33.5 velocity=16 -> lower=-0.802851455917 upper=0.802851455917 effort=20 velocity=52.4
- joint FR_hip_joint: limit lower=-0.802851455917 upper=0.802851455917 effort=33.5 velocity=16 -> lower=-0.802851455917 upper=0.802851455917 effort=20 velocity=52.4
- joint RL_hip_joint: limit lower=-0.802851455917 upper=0.802851455917 effort=33.5 velocity=16 -> lower=-0.802851455917 upper=0.802851455917 effort=20 velocity=52.4
- joint RR_hip_joint: limit lower=-0.802851455917 upper=0.802851455917 effort=33.5 velocity=16 -> lower=-0.802851455917 upper=0.802851455917 effort=20 velocity=52.4
